Commit message: change name controller add imu hardware

File: src/agv_description/ros2_control/agv_system.ros2_control.xacro (robot description, xacro)
@@ -1,26 +1,38 @@
 <?xml version="1.0"?>
 <robot xmlns:xacro="http://www.ros.org/wiki/xacro">
-  <xacro:macro name="agv_system" params="name prefix use_fake_hardware:=^|false user_real_hardware:=^|false slowdown:=2.0">
-    <ros2_control name="${name}" type="system">
+  <xacro:macro name="agv_ros2_control_system" params="prefix">
+    <ros2_control name="imu" type="sensor">
       <hardware>
-        <xacro:if value="${use_fake_hardware}">
-          <plugin>fake_components/GenericSystem</plugin>
-          <param name="fake_sensor_commands">${fake_sensor_commands}</param>
-          <param name="state_following_offset">0.0</param>
-        </xacro:if>
-        <xacro:unless value="${use_fake_hardware}">
-          <plugin>agv_hardware/AGVHardware</plugin>
-          <param name="left_wheel_name">left_wheel_joint</param>
-          <param name="right_wheel_name">right_wheel_joint</param>
-          <param name="loop_rate">30</param>
-          <param name="device">/dev/ttyACM0</param>
-          <param name="baud_rate">115200</param>
-          <param name="timeout_ms">1000</param>
-          <param name="enc_counts_per_rev">220</param>
-          <param name="pid_p">0</param>
-          <param name="pid_d">0</param>
-          <param name="pid_i">0</param>
-          <param name="pid_o">0</param>
-        </xacro:unless>
+        <plugin>imu_hardware/IMUHardware</plugin>
+        <param name="connection_timeout_ms">120000</param>
+        <param name="connection_check_period_ms">500</param>
+      </hardware>
+      <sensor name="imu_joint">
+        <state_interface name="orientation.x" />
+        <state_interface name="orientation.y" />
+        <state_interface name="orientation.z" />
+        <state_interface name="orientation.w" />
+        <state_interface name="angular_velocity.x" />
+        <state_interface name="angular_velocity.y" />
+        <state_interface name="angular_velocity.z" />
+        <state_interface name="linear_acceleration.x" />
+        <state_interface name="linear_acceleration.y" />
+        <state_interface name="linear_acceleration.z" />
+      </sensor>
+    </ros2_control>
+    <ros2_control name="wheels" type="system">
+      <hardware>
+        <plugin>agv_hardware/AGVHardware</plugin>
+        <param name="left_wheel_name">left_wheel_joint</param>
+        <param name="right_wheel_name">right_wheel_joint</param>
+        <param name="loop_rate">30</param>
+        <param name="device">/dev/ttyACM0</param>
+        <param name="baud_rate">115200</param>
+        <param name="timeout_ms">1000</param>
+        <param name="enc_counts_per_rev">220</param>
+        <param name="pid_p">0</param>
+        <param name="pid_d">0</param>
+        <param name="pid_i">0</param>
+        <param name="pid_o">0</param>
       </hardware>
       <joint name="left_wheel_joint">

File: src/agv_description/urdf/agv.urdf.xacro (robot description, xacro)
@@ -1,6 +1,6 @@
 <?xml version="1.0"?>
 <robot xmlns:xacro="http://www.ros.org/wiki/xacro">
-  <xacro:macro name="agv" params="prefix">
-<link
+  <xacro:macro name="agv_system" params="prefix">
+  <link
     name="base_footprint">
     <inertial>

File: src/agv_description/urdf/agv_system.urdf.xacro (robot description, xacro)
@@ -6,8 +6,8 @@
 -->
 <robot xmlns:xacro="http://www.ros.org/wiki/xacro" name="agv_robot">
-  <xacro:arg name="use_sim" default="false" />
+  <!-- <xacro:arg name="use_sim" default="false" /> -->
   <!-- Enable setting arguments from the launch file -->
-  <xacro:arg name="use_fake_hardware" default="false" />
-  <xacro:arg name="user_real_hardware" default="true" />
+  <!-- <xacro:arg name="use_fake_hardware" default="false" />
+  <xacro:arg name="user_real_hardware" default="true" /> -->
   <xacro:arg name="prefix" default="" />
   <xacro:include filename="$(find agv_description)/urdf/agv.urdf.xacro" />
@@ -18,9 +18,10 @@
   <!-- Import diffbot ros2_control description -->
   <xacro:include filename="$(find agv_description)/ros2_control/agv_system.ros2_control.xacro" />
-  <xacro:agv prefix="$(arg prefix)" />
+  <xacro:agv_system prefix="$(arg prefix)" />
+  <xacro:agv_ros2_control_system prefix="$(arg prefix)" />
   <!-- <xacro:agv_gazebo prefix="$(arg prefix)" /> -->
-  <xacro:agv_system
+  <!-- <xacro:agv_system
     name="AGVSystem" prefix="$(arg prefix)"
     use_fake_hardware="$(arg use_fake_hardware)"
-    user_real_hardware="$(arg user_real_hardware)"/>
+    user_real_hardware="$(arg user_real_hardware)"/> -->
 </robot>
