Commit message: change name of nbot hardware

File: src/nbot_description/ros2_control/nbot_diff_system.ros2_control.xacro (robot description, xacro)
@@ -1,8 +1,8 @@
 <?xml version="1.0"?>
 <robot xmlns:xacro="http://www.ros.org/wiki/xacro">
-  <xacro:macro name="agv_ros2_control_system" params="prefix">
+  <xacro:macro name="nbot_ros2_control_system" params="prefix">
     <ros2_control name="imu" type="sensor">
       <hardware>
-        <plugin>nbot_hardware/NbotImuSensor</plugin>
+        <plugin>nbot_hardware_interfaces/NbotImuSensor</plugin>
         <param name="connection_timeout_ms">120000</param>
         <param name="connection_check_period_ms">500</param>
@@ -23,5 +23,5 @@
     <ros2_control name="wheels" type="system">
       <hardware>
-        <plugin>nbot_hardware/NbotWheelsController</plugin>
+        <plugin>nbot_hardware_interfaces/NbotWheelsController</plugin>
         <param name="left_wheel_name">left_wheel_joint</param>
         <param name="right_wheel_name">right_wheel_joint</param>

File: src/nbot_description/urdf/nbot_diff_system.urdf.xacro (robot description, xacro)
@@ -11,5 +11,5 @@
   <xacro:arg name="user_real_hardware" default="true" /> -->
   <xacro:arg name="prefix" default="" />
-  <xacro:include filename="$(find agv_description)/urdf/nbot_base.urdf.xacro" />
+  <xacro:include filename="$(find nbot_description)/urdf/nbot_base.urdf.xacro" />
   <!-- Import all Gazebo-customization elements, including Gazebo colors -->
   <!-- <xacro:include filename="$(find agv_description)/gazebo/agv.gazebo.xacro" /> -->
@@ -17,7 +17,7 @@
   <!-- <xacro:include filename="$(find agv_description)/gazebo/agv.materials.xacro" /> -->
   <!-- Import diffbot ros2_control description -->
-  <xacro:include filename="$(find agv_description)/ros2_control/nbot_diff_system.ros2_control.xacro" />
+  <xacro:include filename="$(find nbot_description)/ros2_control/nbot_diff_system.ros2_control.xacro" />
   <xacro:agv_system prefix="$(arg prefix)" />
-  <xacro:agv_ros2_control_system prefix="$(arg prefix)" />
+  <xacro:nbot_ros2_control_system prefix="$(arg prefix)" />
   <!-- <xacro:agv_gazebo prefix="$(arg prefix)" /> -->
   <!-- <xacro:agv_system
